Commit message: ! fixed relative paths in URDFs ! updated README.md

File: my_ur5_description/urdf/myur5_gripper.urdf.xacro (robot description, xacro)
@@ -84,5 +84,5 @@
         <visual>
         <geometry>
-            <mesh filename="package://robotiq_description/meshes/robotiq_85_coupler.stl" />
+            <mesh filename="file://$(find robotiq_description)/meshes/robotiq_85_coupler.stl" />
         </geometry>
         <material name="flat_black"/>
@@ -90,5 +90,5 @@
         <collision>
         <geometry>
-            <mesh filename="package://robotiq_description/meshes/robotiq_85_coupler.stl" />
+            <mesh filename="file://$(find robotiq_description)/meshes/robotiq_85_coupler.stl" />
         </geometry>
         </collision>

File: robotiq/robotiq_description/urdf/robotiq_85_gripper.urdf.xacro (robot description, xacro)
@@ -11,10 +11,10 @@
       <visual>
         <geometry>
-          <mesh filename="package://robotiq_description/meshes/visual/robotiq_85_base_link.dae"/>
-        </geometry>
-      </visual>
-      <collision>
-        <geometry>
-          <mesh filename="package://robotiq_description/meshes/collision/robotiq_85_base_link.stl"/>
+          <mesh filename="file://$(find robotiq_description)/meshes/visual/robotiq_85_base_link.dae"/>
+        </geometry>
+      </visual>
+      <collision>
+        <geometry>
+          <mesh filename="file://$(find robotiq_description)/meshes/collision/robotiq_85_base_link.stl"/>
         </geometry>
       </collision>
@@ -45,10 +45,10 @@
       <visual>
         <geometry>
-          <mesh filename="package://robotiq_description/meshes/visual/robotiq_85_knuckle_link.dae"/>
-        </geometry>
-      </visual>
-      <collision>
-        <geometry>
-          <mesh filename="package://robotiq_description/meshes/collision/robotiq_85_knuckle_link.stl"/>
+          <mesh filename="file://$(find robotiq_description)/meshes/visual/robotiq_85_knuckle_link.dae"/>
+        </geometry>
+      </visual>
+      <collision>
+        <geometry>
+          <mesh filename="file://$(find robotiq_description)/meshes/collision/robotiq_85_knuckle_link.stl"/>
         </geometry>
       </collision>
@@ -64,10 +64,10 @@
       <visual>
         <geometry>
-          <mesh filename="package://robotiq_description/meshes/visual/robotiq_85_knuckle_link.dae"/>
-        </geometry>
-      </visual>
-      <collision>
-        <geometry>
-          <mesh filename="package://robotiq_description/meshes/collision/robotiq_85_knuckle_link.stl"/>
+          <mesh filename="file://$(find robotiq_description)/meshes/visual/robotiq_85_knuckle_link.dae"/>
+        </geometry>
+      </visual>
+      <collision>
+        <geometry>
+          <mesh filename="file://$(find robotiq_description)/meshes/collision/robotiq_85_knuckle_link.stl"/>
         </geometry>
       </collision>
@@ -93,10 +93,10 @@
       <visual>
         <geometry>
-          <mesh filename="package://robotiq_description/meshes/visual/robotiq_85_finger_link.dae"/>
-        </geometry>
-      </visual>
-      <collision>
-        <geometry>
-          <mesh filename="package://robotiq_description/meshes/collision/robotiq_85_finger_link.stl"/>
+          <mesh filename="file://$(find robotiq_description)/meshes/visual/robotiq_85_finger_link.dae"/>
+        </geometry>
+      </visual>
+      <collision>
+        <geometry>
+          <mesh filename="file://$(find robotiq_description)/meshes/collision/robotiq_85_finger_link.stl"/>
         </geometry>
       </collision>
@@ -112,10 +112,10 @@
       <visual>
         <geometry>
-          <mesh filename="package://robotiq_description/meshes/visual/robotiq_85_finger_link.dae"/>
-        </geometry>
-      </visual>
-      <collision>
-        <geometry>
-          <mesh filename="package://robotiq_description/meshes/collision/robotiq_85_finger_link.stl"/>
+          <mesh filename="file://$(find robotiq_description)/meshes/visual/robotiq_85_finger_link.dae"/>
+        </geometry>
+      </visual>
+      <collision>
+        <geometry>
+          <mesh filename="file://$(find robotiq_description)/meshes/collision/robotiq_85_finger_link.stl"/>
         </geometry>
       </collision>
@@ -147,10 +147,10 @@
       <visual>
         <geometry>
-          <mesh filename="package://robotiq_description/meshes/visual/robotiq_85_inner_knuckle_link.dae"/>
-        </geometry>
-      </visual>
-      <collision>
-        <geometry>
-          <mesh filename="package://robotiq_description/meshes/collision/robotiq_85_inner_knuckle_link.stl"/>
+          <mesh filename="file://$(find robotiq_description)/meshes/visual/robotiq_85_inner_knuckle_link.dae"/>
+        </geometry>
+      </visual>
+      <collision>
+        <geometry>
+          <mesh filename="file://$(find robotiq_description)/meshes/collision/robotiq_85_inner_knuckle_link.stl"/>
         </geometry>
       </collision>
@@ -166,10 +166,10 @@
       <visual>
         <geometry>
-          <mesh filename="package://robotiq_description/meshes/visual/robotiq_85_inner_knuckle_link.dae"/>
-        </geometry>
-      </visual>
-      <collision>
-        <geometry>
-          <mesh filename="package://robotiq_description/meshes/collision/robotiq_85_inner_knuckle_link.stl"/>
+          <mesh filename="file://$(find robotiq_description)/meshes/visual/robotiq_85_inner_knuckle_link.dae"/>
+        </geometry>
+      </visual>
+      <collision>
+        <geometry>
+          <mesh filename="file://$(find robotiq_description)/meshes/collision/robotiq_85_inner_knuckle_link.stl"/>
         </geometry>
       </collision>
@@ -201,10 +201,10 @@
       <visual>
         <geometry>
-          <mesh filename="package://robotiq_description/meshes/visual/robotiq_85_finger_tip_link.dae"/>
-        </geometry>
-      </visual>
-      <collision>
-        <geometry>
-          <mesh filename="package://robotiq_description/meshes/collision/robotiq_85_finger_tip_link.stl"/>
+          <mesh filename="file://$(find robotiq_description)/meshes/visual/robotiq_85_finger_tip_link.dae"/>
+        </geometry>
+      </visual>
+      <collision>
+        <geometry>
+          <mesh filename="file://$(find robotiq_description)/meshes/collision/robotiq_85_finger_tip_link.stl"/>
         </geometry>
       </collision>
@@ -220,10 +220,10 @@
       <visual>
         <geometry>
-          <mesh filename="package://robotiq_description/meshes/visual/robotiq_85_finger_tip_link.dae"/>
-        </geometry>
-      </visual>
-      <collision>
-        <geometry>
-          <mesh filename="package://robotiq_description/meshes/collision/robotiq_85_finger_tip_link.stl"/>
+          <mesh filename="file://$(find robotiq_description)/meshes/visual/robotiq_85_finger_tip_link.dae"/>
+        </geometry>
+      </visual>
+      <collision>
+        <geometry>
+          <mesh filename="file://$(find robotiq_description)/meshes/collision/robotiq_85_finger_tip_link.stl"/>
         </geometry>
       </collision>

File: ur5e_gripper_moveit_config/config/gazebo_ur5e_robot.urdf (robot description, URDF)
Before this commit: robot ur5e_robot, 23 links, 22 joints
Links:
- link base_link_inertia: geometry collision mesh filename=$(find ur_description)/meshes/ur5e/collision/base.stl; visual mesh filename=$(find ur_description)/meshes/ur5e/visual/base.dae
- link forearm_link: geometry collision mesh filename=$(find ur_description)/meshes/ur5e/collision/forearm.stl; visual mesh filename=$(find ur_description)/meshes/ur5e/visual/forearm.dae
- link robotiq_85_base_link: geometry collision mesh filename=$(find robotiq_description)/meshes/collision/robotiq_85_bas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; visual mesh filename=$(find robotiq_description)/meshes/visual/robotiq_85_base_l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
- link robotiq_85_left_finger_link: geometry collision mesh filename=$(find robotiq_description)/meshes/collision/robotiq_85_fin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; visual mesh filename=$(find robotiq_description)/meshes/visual/robotiq_85_finger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
- link robotiq_85_left_finger_tip_link: geometry collision mesh filename=$(find robotiq_description)/meshes/collision/robotiq_85_fin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; visual mesh filename=$(find robotiq_description)/meshes/visual/robotiq_85_finger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
- link robotiq_85_left_inner_knuckle_link: geometry collision mesh filename=$(find robotiq_description)/meshes/collision/robotiq_85_inn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; visual mesh filename=$(find robotiq_description)/meshes/visual/robotiq_85_inner_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
- link robotiq_85_left_knuckle_link: geometry collision mesh filename=$(find robotiq_description)/meshes/collision/robotiq_85_knu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; visual mesh filename=$(find robotiq_description)/meshes/visual/robotiq_85_knuckl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
- link robotiq_85_right_finger_link: geometry collision mesh filename=$(find robotiq_description)/meshes/collision/robotiq_85_fin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; visual mesh filename=$(find robotiq_description)/meshes/visual/robotiq_85_finger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
- link robotiq_85_right_finger_tip_link: geometry collision mesh filename=$(find robotiq_description)/meshes/collision/robotiq_85_fin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; visual mesh filename=$(find robotiq_description)/meshes/visual/robotiq_85_finger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
- link robotiq_85_right_inner_knuckle_link: geometry collision mesh filename=$(find robotiq_description)/meshes/collision/robotiq_85_inn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; visual mesh filename=$(find robotiq_description)/meshes/visual/robotiq_85_inner_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
- link robotiq_85_right_knuckle_link: geometry collision mesh filename=$(find robotiq_description)/meshes/collision/robotiq_85_knu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; visual mesh filename=$(find robotiq_description)/meshes/visual/robotiq_85_knuckl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
- link robotiq_coupler: geometry collision mesh filename=file://$(find robotiq_description)/meshes/robotiq_85_couple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; visual mesh filename=file://$(find robotiq_description)/meshes/robotiq_85_couple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
- link shoulder_link: geometry collision mesh filename=$(find ur_description)/meshes/ur5e/collision/shoulder.stl; visual mesh filename=$(find ur_description)/meshes/ur5e/visual/shoulder.dae
- link upper_arm_link: geometry collision mesh filename=$(find ur_description)/meshes/ur5e/collision/upperarm.stl; visual mesh filename=$(find ur_description)/meshes/ur5e/visual/upperarm.dae
- link wrist_1_link: geometry collision mesh filename=$(find ur_description)/meshes/ur5e/collision/wrist1.stl; visual mesh filename=$(find ur_description)/meshes/ur5e/visual/wrist1.dae
- link wrist_2_link: geometry collision mesh filename=$(find ur_description)/meshes/ur5e/collision/wrist2.stl; visual mesh filename=$(find ur_description)/meshes/ur5e/visual/wrist2.dae
- link wrist_3_link: geometry collision mesh filename=$(find ur_description)/meshes/ur5e/collision/wrist3.stl; visual mesh filename=$(find ur_description)/meshes/ur5e/visual/wrist3.dae

File: urdf/myur5_gripper.urdf.xacro (robot description, xacro)
@@ -84,5 +84,5 @@
         <visual>
         <geometry>
-            <mesh filename="package://robotiq_description/meshes/robotiq_85_coupler.stl" />
+            <mesh filename="file://$(find robotiq_description)/meshes/robotiq_85_coupler.stl" />
         </geometry>
         <material name="flat_black"/>
@@ -90,5 +90,5 @@
         <collision>
         <geometry>
-            <mesh filename="package://robotiq_description/meshes/robotiq_85_coupler.stl" />
+            <mesh filename="file://$(find robotiq_description)/meshes/robotiq_85_coupler.stl" />
         </geometry>
         </collision>
